File: Opentrons_smoothieboard-5driver.brd (EAGLE design)
At the start: 129.6 x 110.9 mm, 385 parts, among them IC1 LPC1769, IC10 LM1117-3.3V, IC11 78L12F, IC12 A4982, IC13 R-78E-5.0, IC14 TC4427, IC15 TC4427, IC2 A4982, IC3 A4982, IC4 MCP44X1, IC5 A4982, IC6 A4982, IC9 MCP44X1, J10 POWER_JACKSMD, Q1 BSL207SP, Q10 SUD50P04-08-GE3, Q2 12MHz, Q3 25MHz, Q4 ZXMN4A06, Q5 AOT240L, Q6 AOT240L, Q7 AOT240L, Q8 ZXMN4A06, Q9 ZXMN4A06, U1 USD-SOCKETNEW, X14 USBPTH

Commit message: adds 6th driver
Parts:
- added C89, C90, C91, C93, C95: .1uF, rcl:C0603
- added C92: .22uF, rcl:C0603
- added C94: 100uF, SparkFun:PANASONIC_E
- added D27, D28, D29, D30: SMBJ16(C)A, My_Lib:DO214-AA_(SMB)
- added IC16: A4982, A4982:ETSSOP24
- added J12: (no value), con-amp:10X05MTA
- added L50, L51, L52, L53, L54, L55, L56: BEAD0603S601A20T, My_Lib:0603(1608)
- added L57, L58: CHOK4525S601A15T, My_Lib:L-4525
- added R109, R110, R114: 10K, resistor:R0603
- added R111, R112: 0.05R, SparkFun:R2512
- added R113: NP, resistor:R0603
Connections:
- new net DIR6: IC16.P14
- new net EN6: IC16.P23
- new net J5_1A1: D27.2, J12.1, L57.4
- new net J5_1B1: D28.2, J12.2, L57.1
- new net J5_2A1: D29.2, J12.3, L58.4
- new net J5_2B1: D30.2, J12.4, L58.1
- new net N$11: C89.2, IC16.P01
- new net N$120: C89.1, IC16.P02
- new net N$169: C90.2, IC16.P03
- new net N$178: IC16.P17, R111.2
- new net N$179: IC16.P20, R112.2
- new net N$180: IC16.P18, L54.2
- new net N$181: IC16.P15, L53.2
- new net N$184: IC16.P19, L55.2
- new net N$185: IC16.P22, L56.2
- new net N$186: IC16.P08, R109.1, R113.1
- new net N$187: C92.2, IC16.P04
- new net N$188: IC16.P09, R110.1
- new net N$189: IC16.P07, R114.1
- new net N$190: C91.1, IC16.P10, L50.1
- new net N$191: IC16.P16, L51.1
- new net N$192: IC16.P21, L52.1
- new net N$193: L54.1, L57.2
- new net N$194: L53.1, L57.3
- new net N$195: L55.1, L58.3
- new net N$196: L56.1, L58.2
- new net PW6: IC16.P12, IC9.9
- new net STP6: IC16.P11
- net 3.3V: now also L50.2, R110.2, R113.2, R114.2
- net GND: now also C91.2, C92.1, C93.2, C94.-, C95.2, D27.1, D28.1, D29.1, D30.1, IC16.EPAD, IC16.P13, IC16.P24, J12.5, R109.2, R111.1, R112.1
- net MS1: now also IC16.P05
- net MS2: now also IC16.P06
- net VBB: now also C90.1, C93.1, C94.+, C95.1, L51.2, L52.2
- net ZETA_CURRENT: no longer IC9.9
Routing:
- net ZETA_CURRENT: track 17.0 -> 16.2 mm
